File: kicad/SCCS-RPI.kicad_sch (KiCad schematic)
At the start: 62 parts, among them J1 Conn_Coaxial, J2 12VDC IN, U1 SN74LVC2T45DCUR, U2 AP64501SP-13

Commit message: Update SCCS-RPI KiCad design and production files
Add GPS RF ESD and matching (ESD103-B1-02EL, 27nH, 10R, 100nF),
swap the 10A fuses to A16-1000, retune copper zone fills, and
regenerate BOM, positions, netlist, gerbers, and schematics PDF.
Parts:
- added C8: 100nF, Capacitor_SMD:C_0805_2012Metric, symbol Device:C_Small
- added D1: ESD103-B1-02EL, Diode_SMD:D_0402_1005Metric, symbol Device:D_TVS
- added L1: 27nH, Inductor_SMD:L_0603_1608Metric, symbol Device:L_Small
- added R8: 10R, Resistor_SMD:R_0805_2012Metric, symbol Device:R
- F1: value 10A -> A16-1000 10A; LCSC Part # C14767 -> C135398
- renumbered C9 to C10, C10 to C11, C11 to C12, C12 to C13, C13 to C14, C14 to C15, C15 to C16, C16 to C17, C17 to C18, C18 to C19, C19 to C20, C20 to C21, C21 to C22, C22 to C23, C23 to C24, C24 to C25, C25 to C26, C26 to C27, C27 to C28, C8 to C9, D1 to D2, D2 to D3, D3 to D4, D4 to D5, D5 to D6, L1 to L2, L2 to L3, R9 to R10, R10 to R11, R11 to R12, R12 to R13, R13 to R14, R14 to R15, R15 to R16, R8 to R9
Connections:
- net GND: now also GPS1.7 (VDD_USB), C8.2, D1.1 (A1)
- net at GPS1.11 (RF_IN), J1.1 (In): now also D1.2 (A2), L1.2
- net at GPS1.9 (VCC_RF): now also C8.1, R8.1
- new net: L1.1, R8.2
- no-connect marks 18 -> 16
Other:
- note added: "RF ESD"
- moved on the sheet: C6, C7, J1

Commit message: Update SCCS-RPI KiCad design and production files
Split 5V and 3V3 regulation onto dedicated Power sheets with a second
AP64501 buck, extra inductor and passives, update the enclosure
bracket, and regenerate BOM, positions, netlist, gerbers, and
schematics PDF.
Parts:
- removed C10, C11, C12, C13, C14, C15, C16, C17: 22uF, Capacitor_SMD:C_0805_2012Metric, symbol Device:C_Small
- removed C18: 2.7nF, Capacitor_SMD:C_0805_2012Metric, symbol Device:C_Small
- removed C26: 33pF, Capacitor_SMD:C_0805_2012Metric, symbol Device:C_Small
- removed C28: 10nF, Capacitor_SMD:C_0805_2012Metric, symbol Device:C_Small
- removed C9: 0.1uF, Capacitor_SMD:C_0805_2012Metric, symbol Device:C_Small
- removed L2: 3.3uH, Inductor_SMD:L_SXN_SMDRI127, symbol Device:L_Small
- removed R12: 15.8K, Resistor_SMD:R_0805_2012Metric, symbol Device:R_Small
- removed R15: 115K, Resistor_SMD:R_0805_2012Metric, symbol Device:R_Small
- removed R16: 22.1K, Resistor_SMD:R_0805_2012Metric, symbol Device:R_Small
- removed U2: AP64501SP-13, Package_SO:SOIC-8-1EP_3.9x4.9mm_P1.27mm_EP2.95x4.9mm_Mask2.71x3.4mm_ThermalVias, symbol CM4IO:AP64351
- renumbered C20 to C10, C21 to C11, C22 to C12, C23 to C13, C24 to C14, C25 to C15, C27 to C16, C19 to C9, L3 to L2, R13 to R12, R14 to R13
Connections:
- net +3V3: no longer PI1.1 (Pin_1)
- net Power - 3V3/Power_in: now reaches C10.2, C11.2, C12.2, C13.2, C14.2, C15.2, C9.1, L2.2, R12.1
- no-connect marks 16 -> 17
Other:
- added sheet Power - 3V3 (power.kicad_sch)
- added sheet Power - 5V (power.kicad_sch)
- note added: "1. Power circuit provides 5V 2. 12V buck (U7 AP64501) provides system 3.3V; Pi 3V3 pins isolated 3. 1-Wire Bus Notes: Board has a 2.2K pull-up on the data line. Put a 220R resistor on the data pin of each temp sensor but ensure it's not in series with the bus. Put a 100nF ceramic cap across VCC and GND at each temp sensor. 4. WS281X RPI Notes: Put a 220uF electrolytic cap between 12V and GND at t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"
- note removed: "1. Power circuit provides 5V 2. RPI Provides 3.3V 3. 1-Wire Bus Notes: Board has a 2.2K pull-up on the data line. Put a 220R resistor on the data pin of each temp sensor but ensure it's not in series with the bus. Put a 100nF ceramic cap across VCC and GND at each temp sensor. 4. WS281X RPI Notes: Put a 220uF electrolytic cap between 12V and GND at the start of each LED strip 5. UARTS: UART1 / GP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"
- note removed: "Put thermal vias below EP pad"
- note removed: "Wire resistors to clean side of output where the caps are"
