File: kicad/analog_inputs.kicad_sch (KiCad schematic)
At the start: 4 parts

Commit message: Update SCCS-RPI KiCad design and production files
Add GPS RF ESD and matching (ESD103-B1-02EL, 27nH, 10R, 100nF),
swap the 10A fuses to A16-1000, retune copper zone fills, and
regenerate BOM, positions, netlist, gerbers, and schematics PDF.
Parts:
- renumbered C29 to C30, R17 to R18
Changed lines of the file:
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@@
 		(in_pos_files yes)
 		(dnp no)
-		(property "Reference" "R17"
+		(property "Reference" "R18"
 			(at 110.49 63.754 90)
 			(show_name no)
@@
 			(project "SCCS-RPI"
 				(path "/ce21946f-7655-4864-b48a-50deff8538eb/11e9aa4c-c1a1-4a8f-a0a0-7141df7ab674"
+					(reference "R19")
+					(unit 1)
+				)
+				(path "/ce21946f-7655-4864-b48a-50deff8538eb/3114b48f-2d53-4033-bb6c-4b7d97201800"
 					(reference "R18")
 					(unit 1)
 				)
-				(path "/ce21946f-7655-4864-b48a-50deff8538eb/3114b48f-2d53-4033-bb6c-4b7d97201800"
-					(reference "R17")
-					(unit 1)
-				)
 				(path "/ce21946f-7655-4864-b48a-50deff8538eb/f275b187-1ecf-4da8-9601-a32837f11b2b"
-					(reference "R19")
+					(reference "R20")
 					(unit 1)
 				)
@@
 		(dnp no)
 		(fields_autoplaced yes)
-		(property "Reference" "C29"
+		(property "Reference" "C30"
 			(at 121.92 72.3962 0)
 			(show_name no)
@@
 			(project "SCCS-RPI"
 				(path "/ce21946f-7655-4864-b48a-50deff8538eb/11e9aa4c-c1a1-4a8f-a0a0-7141df7ab674"
+					(reference "C31")
+					(unit 1)
+				)
+				(path "/ce21946f-7655-4864-b48a-50deff8538eb/3114b48f-2d53-4033-bb6c-4b7d97201800"
 					(reference "C30")
 					(unit 1)
 				)
-				(path "/ce21946f-7655-4864-b48a-50deff8538eb/3114b48f-2d53-4033-bb6c-4b7d97201800"
-					(reference "C29")
-					(unit 1)
-				)
 				(path "/ce21946f-7655-4864-b48a-50deff8538eb/f275b187-1ecf-4da8-9601-a32837f11b2b"
-					(reference "C31")
-					(unit 1)
-				)
+					(reference "C32")
+					(unit 1)
+				)

Commit message: Update SCCS-RPI KiCad design and production files
Split 5V and 3V3 regulation onto dedicated Power sheets with a second
AP64501 buck, extra inductor and passives, update the enclosure
bracket, and regenerate BOM, positions, netlist, gerbers, and
schematics PDF.
Parts:
- renumbered C30 to C18, R18 to R15
Changed lines of the file:
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@@
 		(in_pos_files yes)
 		(dnp no)
-		(property "Reference" "R18"
+		(property "Reference" "R15"
 			(at 110.49 63.754 90)
 			(show_name no)
@@
 			(project "SCCS-RPI"
 				(path "/ce21946f-7655-4864-b48a-50deff8538eb/11e9aa4c-c1a1-4a8f-a0a0-7141df7ab674"
-					(reference "R19")
+					(reference "R16")
 					(unit 1)
 				)
 				(path "/ce21946f-7655-4864-b48a-50deff8538eb/3114b48f-2d53-4033-bb6c-4b7d97201800"
-					(reference "R18")
+					(reference "R15")
 					(unit 1)
 				)
 				(path "/ce21946f-7655-4864-b48a-50deff8538eb/f275b187-1ecf-4da8-9601-a32837f11b2b"
-					(reference "R20")
+					(reference "R17")
 					(unit 1)
 				)
@@
 		(dnp no)
 		(fields_autoplaced yes)
-		(property "Reference" "#PWR034"
+		(property "Reference" "#PWR033"
 			(at 99.06 85.09 0)
 			(hide yes)
@@
 			(project "SCCS-RPI"
 				(path "/ce21946f-7655-4864-b48a-50deff8538eb/11e9aa4c-c1a1-4a8f-a0a0-7141df7ab674"
-					(reference "#PWR036")
+					(reference "#PWR035")
 					(unit 1)
 				)
 				(path "/ce21946f-7655-4864-b48a-50deff8538eb/3114b48f-2d53-4033-bb6c-4b7d97201800"
-					(reference "#PWR034")
+					(reference "#PWR033")
 					(unit 1)
 				)
 				(path "/ce21946f-7655-4864-b48a-50deff8538eb/f275b187-1ecf-4da8-9601-a32837f11b2b"
-					(reference "#PWR038")
+					(reference "#PWR037")
 					(unit 1)
 				)
@@
 		(dnp no)
 		(fields_autoplaced yes)
-		(property "Reference" "C30"
+		(property "Reference" "C18"
 			(at 121.92 72.3962 0)
 			(show_name no)
@@
 			(project "SCCS-RPI"
 				(path "/ce21946f-7655-4864-b48a-50deff8538eb/11e9aa4c-c1a1-4a8f-a0a0-7141df7ab674"
-					(reference "C31")
+					(reference "C19")
 					(unit 1)
 				)
 				(path "/ce21946f-7655-4864-b48a-50deff8538eb/3114b48f-2d53-4033-bb6c-4b7d97201800"
-					(reference "C30")
+					(reference "C18")
 					(unit 1)
 				)
 				(path "/ce21946f-7655-4864-b48a-50deff8538eb/f275b187-1ecf-4da8-9601-a32837f11b2b"
-					(reference "C32")
+					(reference "C20")
 					(unit 1)
 				)
@@
 		(in_pos_files yes)
 		(dnp no)
-		(property "Reference" "#PWR033"
+		(property "Reference" "#PWR032"
 			(at 99.06 66.04 0)
 			(hide yes)
@@
 			(project "SCCS-RPI"
 				(path "/ce21946f-7655-4864-b48a-50deff8538eb/11e9aa4c-c1a1-4a8f-a0a0-7141df7ab674"
-					(reference "#PWR035")
+					(reference "#PWR034")
 					(unit 1)
 				)
 				(path "/ce21946f-7655-4864-b48a-50deff8538eb/3114b48f-2d53-4033-bb6c-4b7d97201800"
-					(reference "#PWR033")
+					(reference "#PWR032")
 					(unit 1)
 				)
 				(path "/ce21946f-7655-4864-b48a-50deff8538eb/f275b187-1ecf-4da8-9601-a32837f11b2b"
-					(reference "#PWR037")
-					(unit 1)
-				)
+					(reference "#PWR036")
+					(unit 1)
+				)
