File: kicad/esp32.kicad_sch (KiCad schematic)
At the start: 9 parts, among them SW1 RESET, SW2 BOOT

Commit message: Update SCCS-RPI KiCad design and production files
Add GPS RF ESD and matching (ESD103-B1-02EL, 27nH, 10R, 100nF),
swap the 10A fuses to A16-1000, retune copper zone fills, and
regenerate BOM, positions, netlist, gerbers, and schematics PDF.
Parts:
- renumbered C48 to C49, C49 to C50, C50 to C51, C51 to C52, R36 to R37, R37 to R38
Changed lines of the file:
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@@
 		(in_pos_files yes)
 		(dnp no)
-		(property "Reference" "C51"
+		(property "Reference" "C52"
 			(at 188.976 89.154 0)
 			(show_name no)
@@
 			(project "SCCS-RPI"
 				(path "/ce21946f-7655-4864-b48a-50deff8538eb/0e54ede7-c3c3-481e-ab9c-f158ab57a6d1"
-					(reference "C51")
-					(unit 1)
-				)
-				(path "/ce21946f-7655-4864-b48a-50deff8538eb/d3b05700-09f1-456c-b82f-4b1205485eff"
-					(reference "C55")
+					(reference "C52")
+					(unit 1)
+				)
+				(path "/ce21946f-7655-4864-b48a-50deff8538eb/d3b05700-09f1-456c-b82f-4b1205485eff"
+					(reference "C56")
 					(unit 1)
 				)
@@
 		(in_pos_files yes)
 		(dnp no)
-		(property "Reference" "R36"
+		(property "Reference" "R37"
 			(at 76.2 56.642 90)
 			(show_name no)
@@
 			(project "SCCS-RPI"
 				(path "/ce21946f-7655-4864-b48a-50deff8538eb/0e54ede7-c3c3-481e-ab9c-f158ab57a6d1"
-					(reference "R36")
-					(unit 1)
-				)
-				(path "/ce21946f-7655-4864-b48a-50deff8538eb/d3b05700-09f1-456c-b82f-4b1205485eff"
-					(reference "R38")
+					(reference "R37")
+					(unit 1)
+				)
+				(path "/ce21946f-7655-4864-b48a-50deff8538eb/d3b05700-09f1-456c-b82f-4b1205485eff"
+					(reference "R39")
 					(unit 1)
 				)
@@
 		(in_pos_files yes)
 		(dnp no)
-		(property "Reference" "C48"
+		(property "Reference" "C49"
 			(at 120.904 45.72 0)
 			(show_name no)
@@
 			(project "SCCS-RPI"
 				(path "/ce21946f-7655-4864-b48a-50deff8538eb/0e54ede7-c3c3-481e-ab9c-f158ab57a6d1"
-					(reference "C48")
-					(unit 1)
-				)
-				(path "/ce21946f-7655-4864-b48a-50deff8538eb/d3b05700-09f1-456c-b82f-4b1205485eff"
-					(reference "C52")
+					(reference "C49")
+					(unit 1)
+				)
+				(path "/ce21946f-7655-4864-b48a-50deff8538eb/d3b05700-09f1-456c-b82f-4b1205485eff"
+					(reference "C53")
 					(unit 1)
 				)
@@
 		(in_pos_files yes)
 		(dnp no)
-		(property "Reference" "R37"
+		(property "Reference" "R38"
 			(at 173.99 76.962 90)
 			(show_name no)
@@
 			(project "SCCS-RPI"
 				(path "/ce21946f-7655-4864-b48a-50deff8538eb/0e54ede7-c3c3-481e-ab9c-f158ab57a6d1"
-					(reference "R37")
-					(unit 1)
-				)
-				(path "/ce21946f-7655-4864-b48a-50deff8538eb/d3b05700-09f1-456c-b82f-4b1205485eff"
-					(reference "R39")
+					(reference "R38")
+					(unit 1)
+				)
+				(path "/ce21946f-7655-4864-b48a-50deff8538eb/d3b05700-09f1-456c-b82f-4b1205485eff"
+					(reference "R40")
 					(unit 1)
 				)
@@
 		(in_pos_files yes)
 		(dnp no)
-		(property "Reference" "C50"
+		(property "Reference" "C51"
 			(at 197.104 86.614 0)
 			(show_name no)
@@
 			(project "SCCS-RPI"
 				(path "/ce21946f-7655-4864-b48a-50deff8538eb/0e54ede7-c3c3-481e-ab9c-f158ab57a6d1"
-					(reference "C50")
-					(unit 1)
-				)
-				(path "/ce21946f-7655-4864-b48a-50deff8538eb/d3b05700-09f1-456c-b82f-4b1205485eff"
-					(reference "C54")
+					(reference "C51")
+					(unit 1)
+				)
+				(path "/ce21946f-7655-4864-b48a-50deff8538eb/d3b05700-09f1-456c-b82f-4b1205485eff"
+					(reference "C55")
 					(unit 1)
 				)
@@
 		(in_pos_files yes)
 		(dnp no)
-		(property "Reference" "C49"
+		(property "Reference" "C50"
 			(at 122.936 45.466 0)
 			(show_name no)
@@
 			(project "SCCS-RPI"
 				(path "/ce21946f-7655-4864-b48a-50deff8538eb/0e54ede7-c3c3-481e-ab9c-f158ab57a6d1"
-					(reference "C49")
-					(unit 1)
-				)
-				(path "/ce21946f-7655-4864-b48a-50deff8538eb/d3b05700-09f1-456c-b82f-4b1205485eff"
-					(reference "C53")
-					(unit 1)
-				)
+					(reference "C50")
+					(unit 1)
+				)
+				(path "/ce21946f-7655-4864-b48a-50deff8538eb/d3b05700-09f1-456c-b82f-4b1205485eff"
+					(reference "C54")
+					(unit 1)
+				)

Commit message: Update SCCS-RPI KiCad design and production files
Split 5V and 3V3 regulation onto dedicated Power sheets with a second
AP64501 buck, extra inductor and passives, update the enclosure
bracket, and regenerate BOM, positions, netlist, gerbers, and
schematics PDF.
Parts:
- renumbered C49 to C37, C50 to C38, C51 to C39, C52 to C40, R37 to R34, R38 to R35
Changed lines of the file:
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@@
 		(in_pos_files yes)
 		(dnp no)
-		(property "Reference" "C52"
+		(property "Reference" "C40"
 			(at 188.976 89.154 0)
 			(show_name no)
@@
 			(project "SCCS-RPI"
 				(path "/ce21946f-7655-4864-b48a-50deff8538eb/0e54ede7-c3c3-481e-ab9c-f158ab57a6d1"
-					(reference "C52")
-					(unit 1)
-				)
-				(path "/ce21946f-7655-4864-b48a-50deff8538eb/d3b05700-09f1-456c-b82f-4b1205485eff"
-					(reference "C56")
+					(reference "C40")
+					(unit 1)
+				)
+				(path "/ce21946f-7655-4864-b48a-50deff8538eb/d3b05700-09f1-456c-b82f-4b1205485eff"
+					(reference "C44")
 					(unit 1)
 				)
@@
 		(in_pos_files yes)
 		(dnp no)
-		(property "Reference" "#PWR061"
+		(property "Reference" "#PWR060"
 			(at 242.57 88.9 0)
 			(hide yes)
@@
 			(project "SCCS-RPI"
 				(path "/ce21946f-7655-4864-b48a-50deff8538eb/0e54ede7-c3c3-481e-ab9c-f158ab57a6d1"
-					(reference "#PWR061")
-					(unit 1)
-				)
-				(path "/ce21946f-7655-4864-b48a-50deff8538eb/d3b05700-09f1-456c-b82f-4b1205485eff"
-					(reference "#PWR070")
+					(reference "#PWR060")
+					(unit 1)
+				)
+				(path "/ce21946f-7655-4864-b48a-50deff8538eb/d3b05700-09f1-456c-b82f-4b1205485eff"
+					(reference "#PWR069")
 					(unit 1)
 				)
@@
 		(in_pos_files yes)
 		(dnp no)
-		(property "Reference" "R37"
+		(property "Reference" "R34"
 			(at 76.2 56.642 90)
 			(show_name no)
@@
 			(project "SCCS-RPI"
 				(path "/ce21946f-7655-4864-b48a-50deff8538eb/0e54ede7-c3c3-481e-ab9c-f158ab57a6d1"
-					(reference "R37")
-					(unit 1)
-				)
-				(path "/ce21946f-7655-4864-b48a-50deff8538eb/d3b05700-09f1-456c-b82f-4b1205485eff"
-					(reference "R39")
+					(reference "R34")
+					(unit 1)
+				)
+				(path "/ce21946f-7655-4864-b48a-50deff8538eb/d3b05700-09f1-456c-b82f-4b1205485eff"
+					(reference "R36")
 					(unit 1)
 				)
@@
 		(in_pos_files yes)
 		(dnp no)
-		(property "Reference" "C49"
+		(property "Reference" "C37"
 			(at 120.904 45.72 0)
 			(show_name no)
@@
 			(project "SCCS-RPI"
 				(path "/ce21946f-7655-4864-b48a-50deff8538eb/0e54ede7-c3c3-481e-ab9c-f158ab57a6d1"
-					(reference "C49")
-					(unit 1)
-				)
-				(path "/ce21946f-7655-4864-b48a-50deff8538eb/d3b05700-09f1-456c-b82f-4b1205485eff"
-					(reference "C53")
+					(reference "C37")
+					(unit 1)
+				)
+				(path "/ce21946f-7655-4864-b48a-50deff8538eb/d3b05700-09f1-456c-b82f-4b1205485eff"
+					(reference "C41")
 					(unit 1)
 				)
@@
 		(dnp no)
 		(fields_autoplaced yes)
-		(property "Reference" "#PWR060"
+		(property "Reference" "#PWR059"
 			(at 185.42 76.2 0)
 			(hide yes)
@@
 			(project "SCCS-RPI"
 				(path "/ce21946f-7655-4864-b48a-50deff8538eb/0e54ede7-c3c3-481e-ab9c-f158ab57a6d1"
-					(reference "#PWR060")
-					(unit 1)
-				)
-				(path "/ce21946f-7655-4864-b48a-50deff8538eb/d3b05700-09f1-456c-b82f-4b1205485eff"
-					(reference "#PWR069")
+					(reference "#PWR059")
+					(unit 1)
+				)
+				(path "/ce21946f-7655-4864-b48a-50deff8538eb/d3b05700-09f1-456c-b82f-4b1205485eff"
+					(reference "#PWR068")
 					(unit 1)
 				)
@@
 		(in_pos_files yes)
 		(dnp no)
-		(property "Reference" "#PWR063"
+		(property "Reference" "#PWR062"
 			(at 121.92 151.13 0)
 			(hide yes)
@@
 			(project "SCCS-RPI"
 				(path "/ce21946f-7655-4864-b48a-50deff8538eb/0e54ede7-c3c3-481e-ab9c-f158ab57a6d1"
-					(reference "#PWR063")
-					(unit 1)
-				)
-				(path "/ce21946f-7655-4864-b48a-50deff8538eb/d3b05700-09f1-456c-b82f-4b1205485eff"
-					(reference "#PWR072")
+					(reference "#PWR062")
+					(unit 1)
+				)
+				(path "/ce21946f-7655-4864-b48a-50deff8538eb/d3b05700-09f1-456c-b82f-4b1205485eff"
+					(reference "#PWR071")
 					(unit 1)
 				)
@@
 		(in_pos_files yes)
 		(dnp no)
-		(property "Reference" "#PWR057"
+		(property "Reference" "#PWR056"
 			(at 127 54.61 0)
 			(hide yes)
@@
 			(project "SCCS-RPI"
 				(path "/ce21946f-7655-4864-b48a-50deff8538eb/0e54ede7-c3c3-481e-ab9c-f158ab57a6d1"
-					(reference "#PWR057")
-					(unit 1)
-				)
-				(path "/ce21946f-7655-4864-b48a-50deff8538eb/d3b05700-09f1-456c-b82f-4b1205485eff"
-					(reference "#PWR066")
+					(reference "#PWR056")
+					(unit 1)
+				)
+				(path "/ce21946f-7655-4864-b48a-50deff8538eb/d3b05700-09f1-456c-b82f-4b1205485eff"
+					(reference "#PWR065")
 					(unit 1)
 				)
@@
 		(in_pos_files yes)
 		(dnp no)
-		(property "Reference" "R38"
+		(property "Reference" "R35"
 			(at 173.99 76.962 90)
 			(show_name no)
@@
 			(project "SCCS-RPI"
 				(path "/ce21946f-7655-4864-b48a-50deff8538eb/0e54ede7-c3c3-481e-ab9c-f158ab57a6d1"
-					(reference "R38")
-					(unit 1)
-				)
-				(path "/ce21946f-7655-4864-b48a-50deff8538eb/d3b05700-09f1-456c-b82f-4b1205485eff"
-					(reference "R40")
+					(reference "R35")
+					(unit 1)
+				)
+				(path "/ce21946f-7655-4864-b48a-50deff8538eb/d3b05700-09f1-456c-b82f-4b1205485eff"
+					(reference "R37")
 					(unit 1)
 				)
@@
 		(in_pos_files yes)
 		(dnp no)
-		(property "Reference" "C51"
+		(property "Reference" "C39"
 			(at 197.104 86.614 0)
 			(show_name no)
@@
 			(project "SCCS-RPI"
 				(path "/ce21946f-7655-4864-b48a-50deff8538eb/0e54ede7-c3c3-481e-ab9c-f158ab57a6d1"
-					(reference "C51")
-					(unit 1)
-				)
-				(path "/ce21946f-7655-4864-b48a-50deff8538eb/d3b05700-09f1-456c-b82f-4b1205485eff"
-					(reference "C55")
+					(reference "C39")
+					(unit 1)
+				)
+				(path "/ce21946f-7655-4864-b48a-50deff8538eb/d3b05700-09f1-456c-b82f-4b1205485eff"
+					(reference "C43")
 					(unit 1)
 				)
@@
 		(in_pos_files yes)
 		(dnp no)
-		(property "Reference" "#PWR055"
+		(property "Reference" "#PWR054"
 			(at 121.92 44.45 0)
 			(hide yes)
@@
 			(project "SCCS-RPI"
 				(path "/ce21946f-7655-4864-b48a-50deff8538eb/0e54ede7-c3c3-481e-ab9c-f158ab57a6d1"
-					(reference "#PWR055")
-					(unit 1)
-				)
-				(path "/ce21946f-7655-4864-b48a-50deff8538eb/d3b05700-09f1-456c-b82f-4b1205485eff"
-					(reference "#PWR064")
+					(reference "#PWR054")
+					(unit 1)
+				)
+				(path "/ce21946f-7655-4864-b48a-50deff8538eb/d3b05700-09f1-456c-b82f-4b1205485eff"
+					(reference "#PWR063")
 					(unit 1)
 				)
@@
 		(in_pos_files yes)
 		(dnp no)
-		(property "Reference" "#PWR056"
+		(property "Reference" "#PWR055"
 			(at 116.84 54.61 0)
 			(hide yes)
@@
 			(project "SCCS-RPI"
 				(path "/ce21946f-7655-4864-b48a-50deff8538eb/0e54ede7-c3c3-481e-ab9c-f158ab57a6d1"
-					(reference "#PWR056")
-					(unit 1)
-				)
-				(path "/ce21946f-7655-4864-b48a-50deff8538eb/d3b05700-09f1-456c-b82f-4b1205485eff"
-					(reference "#PWR065")
+					(reference "#PWR055")
+					(unit 1)
+				)
+				(path "/ce21946f-7655-4864-b48a-50deff8538eb/d3b05700-09f1-456c-b82f-4b1205485eff"
+					(reference "#PWR064")
 					(unit 1)
 				)
@@
 		(dnp no)
 		(fields_autoplaced yes)
-		(property "Reference" "#PWR058"
+		(property "Reference" "#PWR057"
 			(at 82.55 55.88 0)
 			(hide yes)
@@
 			(project "SCCS-RPI"
 				(path "/ce21946f-7655-4864-b48a-50deff8538eb/0e54ede7-c3c3-481e-ab9c-f158ab57a6d1"
-					(reference "#PWR058")
-					(unit 1)
-				)
-				(path "/ce21946f-7655-4864-b48a-50deff8538eb/d3b05700-09f1-456c-b82f-4b1205485eff"
-					(reference "#PWR067")
+					(reference "#PWR057")
+					(unit 1)
+				)
+				(path "/ce21946f-7655-4864-b48a-50deff8538eb/d3b05700-09f1-456c-b82f-4b1205485eff"
+					(reference "#PWR066")
 					(unit 1)
 				)
@@
 		(in_pos_files yes)
 		(dnp no)
-		(property "Reference" "#PWR062"
+		(property "Reference" "#PWR061"
 			(at 189.23 99.06 0)
 			(hide yes)
@@
 			(project "SCCS-RPI"
 				(path "/ce21946f-7655-4864-b48a-50deff8538eb/0e54ede7-c3c3-481e-ab9c-f158ab57a6d1"
-					(reference "#PWR062")
-					(unit 1)
-				)
-				(path "/ce21946f-7655-4864-b48a-50deff8538eb/d3b05700-09f1-456c-b82f-4b1205485eff"
-					(reference "#PWR071")
+					(reference "#PWR061")
+					(unit 1)
+				)
+				(path "/ce21946f-7655-4864-b48a-50deff8538eb/d3b05700-09f1-456c-b82f-4b1205485eff"
+					(reference "#PWR070")
 					(unit 1)
 				)
@@
 		(in_pos_files yes)
 		(dnp no)
-		(property "Reference" "#PWR059"
+		(property "Reference" "#PWR058"
 			(at 59.69 73.66 0)
 			(hide yes)
@@
 			(project "SCCS-RPI"
 				(path "/ce21946f-7655-4864-b48a-50deff8538eb/0e54ede7-c3c3-481e-ab9c-f158ab57a6d1"
-					(reference "#PWR059")
-					(unit 1)
-				)
-				(path "/ce21946f-7655-4864-b48a-50deff8538eb/d3b05700-09f1-456c-b82f-4b1205485eff"
-					(reference "#PWR068")
+					(reference "#PWR058")
+					(unit 1)
+				)
+				(path "/ce21946f-7655-4864-b48a-50deff8538eb/d3b05700-09f1-456c-b82f-4b1205485eff"
+					(reference "#PWR067")
 					(unit 1)
 				)
@@
 		(in_pos_files yes)
 		(dnp no)
-		(property "Reference" "C50"
+		(property "Reference" "C38"
 			(at 122.936 45.466 0)
 			(show_name no)
@@
 			(project "SCCS-RPI"
 				(path "/ce21946f-7655-4864-b48a-50deff8538eb/0e54ede7-c3c3-481e-ab9c-f158ab57a6d1"
-					(reference "C50")
-					(unit 1)
-				)
-				(path "/ce21946f-7655-4864-b48a-50deff8538eb/d3b05700-09f1-456c-b82f-4b1205485eff"
-					(reference "C54")
-					(unit 1)
-				)
+					(reference "C38")
+					(unit 1)
+				)
+				(path "/ce21946f-7655-4864-b48a-50deff8538eb/d3b05700-09f1-456c-b82f-4b1205485eff"
+					(reference "C42")
+					(unit 1)
+				)
