File: kicad/led_channel.kicad_sch (KiCad schematic)
At the start: 5 parts, among them Q1 IRLR7843

Commit message: Update SCCS-RPI KiCad design and production files
Add GPS RF ESD and matching (ESD103-B1-02EL, 27nH, 10R, 100nF),
swap the 10A fuses to A16-1000, retune copper zone fills, and
regenerate BOM, positions, netlist, gerbers, and schematics PDF.
Parts:
- renumbered D19 to D20, R40 to R41, R41 to R42, R42 to R43

Commit message: Update SCCS-RPI KiCad design and production files
Split 5V and 3V3 regulation onto dedicated Power sheets with a second
AP64501 buck, extra inductor and passives, update the enclosure
bracket, and regenerate BOM, positions, netlist, gerbers, and
schematics PDF.
Parts:
- renumbered R41 to R38, R42 to R39, R43 to R40
