File: kicad/relay_channel.kicad_sch (KiCad schematic)
At the start: 12 parts, among them K1 Relay_SPDT, Q17 2N7000, U3 PC817

Commit message: Update SCCS-RPI KiCad design and production files
Add GPS RF ESD and matching (ESD103-B1-02EL, 27nH, 10R, 100nF),
swap the 10A fuses to A16-1000, retune copper zone fills, and
regenerate BOM, positions, netlist, gerbers, and schematics PDF.
Parts:
- F2: value 10A -> A16-1000 10A; LCSC Part # C14767 -> C135398
- renumbered C64 to C65, D37 to D38, D38 to D39, R90 to R91, R91 to R92, R92 to R93, R93 to R94
Changed lines of the file:
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@@
 		(dnp no)
 		(fields_autoplaced yes)
-		(property "Reference" "C64"
+		(property "Reference" "C65"
 			(at 102.8763 39.37 90)
 			(show_name no)
@@
 			(project "SCCS-RPI"
 				(path "/ce21946f-7655-4864-b48a-50deff8538eb/67cc456c-a1bb-42f9-9e79-f18883d18275"
+					(reference "C68")
+					(unit 1)
+				)
+				(path "/ce21946f-7655-4864-b48a-50deff8538eb/6d499a9e-12be-48c7-97b5-aaa8433b7610"
 					(reference "C67")
 					(unit 1)
 				)
-				(path "/ce21946f-7655-4864-b48a-50deff8538eb/6d499a9e-12be-48c7-97b5-aaa8433b7610"
+				(path "/ce21946f-7655-4864-b48a-50deff8538eb/b2c53e19-e42b-4380-a3f5-c04d8b1a12f2"
+					(reference "C65")
+					(unit 1)
+				)
+				(path "/ce21946f-7655-4864-b48a-50deff8538eb/f5b14127-5321-4517-88f3-03b8eaf90121"
 					(reference "C66")
-					(unit 1)
-				)
-				(path "/ce21946f-7655-4864-b48a-50deff8538eb/b2c53e19-e42b-4380-a3f5-c04d8b1a12f2"
-					(reference "C64")
-					(unit 1)
-				)
-				(path "/ce21946f-7655-4864-b48a-50deff8538eb/f5b14127-5321-4517-88f3-03b8eaf90121"
-					(reference "C65")
 					(unit 1)
 				)
@@
 		(in_pos_files yes)
 		(dnp no)
-		(property "Reference" "R93"
+		(property "Reference" "R94"
 			(at 85.09 63.246 90)
 			(show_name no)
@@
 			(project "SCCS-RPI"
 				(path "/ce21946f-7655-4864-b48a-50deff8538eb/67cc456c-a1bb-42f9-9e79-f18883d18275"
-					(reference "R105")
+					(reference "R106")
 					(unit 1)
 				)
 				(path "/ce21946f-7655-4864-b48a-50deff8538eb/6d499a9e-12be-48c7-97b5-aaa8433b7610"
-					(reference "R101")
+					(reference "R102")
 					(unit 1)
 				)
 				(path "/ce21946f-7655-4864-b48a-50deff8538eb/b2c53e19-e42b-4380-a3f5-c04d8b1a12f2"
-					(reference "R93")
+					(reference "R94")
 					(unit 1)
 				)
 				(path "/ce21946f-7655-4864-b48a-50deff8538eb/f5b14127-5321-4517-88f3-03b8eaf90121"
-					(reference "R97")
+					(reference "R98")
 					(unit 1)
 				)
@@
 		(in_pos_files yes)
 		(dnp no)
-		(property "Reference" "R92"
+		(property "Reference" "R93"
 			(at 99.06 56.134 90)
 			(show_name no)
@@
 			(project "SCCS-RPI"
 				(path "/ce21946f-7655-4864-b48a-50deff8538eb/67cc456c-a1bb-42f9-9e79-f18883d18275"
-					(reference "R104")
+					(reference "R105")
 					(unit 1)
 				)
 				(path "/ce21946f-7655-4864-b48a-50deff8538eb/6d499a9e-12be-48c7-97b5-aaa8433b7610"
-					(reference "R100")
+					(reference "R101")
 					(unit 1)
 				)
 				(path "/ce21946f-7655-4864-b48a-50deff8538eb/b2c53e19-e42b-4380-a3f5-c04d8b1a12f2"
-					(reference "R92")
+					(reference "R93")
 					(unit 1)
 				)
 				(path "/ce21946f-7655-4864-b48a-50deff8538eb/f5b14127-5321-4517-88f3-03b8eaf90121"
-					(reference "R96")
+					(reference "R97")
 					(unit 1)
 				)
@@
 		(in_pos_files yes)
 		(dnp no)
-		(property "Reference" "D37"
+		(property "Reference" "D38"
 			(at 129.286 51.562 0)
 			(show_name no)
@@
 			(project "SCCS-RPI"
 				(path "/ce21946f-7655-4864-b48a-50deff8538eb/67cc456c-a1bb-42f9-9e79-f18883d18275"
-					(reference "D43")
+					(reference "D44")
 					(unit 1)
 				)
 				(path "/ce21946f-7655-4864-b48a-50deff8538eb/6d499a9e-12be-48c7-97b5-aaa8433b7610"
-					(reference "D41")
+					(reference "D42")
 					(unit 1)
 				)
 				(path "/ce21946f-7655-4864-b48a-50deff8538eb/b2c53e19-e42b-4380-a3f5-c04d8b1a12f2"
-					(reference "D37")
+					(reference "D38")
 					(unit 1)
 				)
 				(path "/ce21946f-7655-4864-b48a-50deff8538eb/f5b14127-5321-4517-88f3-03b8eaf90121"
-					(reference "D39")
+					(reference "D40")
 					(unit 1)
 				)
@@
 		(in_pos_files yes)
 		(dnp no)
-		(property "Reference" "R90"
+		(property "Reference" "R91"
 			(at 63.5 48.006 90)
 			(show_name no)
@@
 			(project "SCCS-RPI"
 				(path "/ce21946f-7655-4864-b48a-50deff8538eb/67cc456c-a1bb-42f9-9e79-f18883d18275"
-					(reference "R102")
+					(reference "R103")
 					(unit 1)
 				)
 				(path "/ce21946f-7655-4864-b48a-50deff8538eb/6d499a9e-12be-48c7-97b5-aaa8433b7610"
-					(reference "R98")
+					(reference "R99")
 					(unit 1)
 				)
 				(path "/ce21946f-7655-4864-b48a-50deff8538eb/b2c53e19-e42b-4380-a3f5-c04d8b1a12f2"
-					(reference "R90")
+					(reference "R91")
 					(unit 1)
 				)
 				(path "/ce21946f-7655-4864-b48a-50deff8538eb/f5b14127-5321-4517-88f3-03b8eaf90121"
-					(reference "R94")
+					(reference "R95")
 					(unit 1)
 				)
@@
 		(in_pos_files yes)
 		(dnp no)
-		(property "Reference" "R91"
+		(property "Reference" "R92"
 			(at 121.92 52.578 90)
 			(show_name no)
@@
 			(project "SCCS-RPI"
 				(path "/ce21946f-7655-4864-b48a-50deff8538eb/67cc456c-a1bb-42f9-9e79-f18883d18275"
-					(reference "R103")
+					(reference "R104")
 					(unit 1)
 				)
 				(path "/ce21946f-7655-4864-b48a-50deff8538eb/6d499a9e-12be-48c7-97b5-aaa8433b7610"
-					(reference "R99")
+					(reference "R100")
 					(unit 1)
 				)
 				(path "/ce21946f-7655-4864-b48a-50deff8538eb/b2c53e19-e42b-4380-a3f5-c04d8b1a12f2"
-					(reference "R91")
+					(reference "R92")
 					(unit 1)
 				)
 				(path "/ce21946f-7655-4864-b48a-50deff8538eb/f5b14127-5321-4517-88f3-03b8eaf90121"
-					(reference "R95")
+					(reference "R96")
 					(unit 1)
 				)
@@
 			)
 		)
-		(property "Value" "10A"
+		(property "Value" "A16-1000 10A"
 			(at 146.05 71.374 90)
 			(show_name no)
@@
 			)
 		)
-		(property "LCSC Part #" "C14767"
+		(property "LCSC Part #" "C135398"
 			(at 146.05 69.85 90)
 			(hide yes)
@@
 		(in_pos_files yes)
 		(dnp no)
-		(property "Reference" "D38"
+		(property "Reference" "D39"
 			(at 121.666 57.658 0)
 			(show_name no)
@@
 			(project "SCCS-RPI"
 				(path "/ce21946f-7655-4864-b48a-50deff8538eb/67cc456c-a1bb-42f9-9e79-f18883d18275"
-					(reference "D44")
+					(reference "D45")
 					(unit 1)
 				)
 				(path "/ce21946f-7655-4864-b48a-50deff8538eb/6d499a9e-12be-48c7-97b5-aaa8433b7610"
-					(reference "D42")
+					(reference "D43")
 					(unit 1)
 				)
 				(path "/ce21946f-7655-4864-b48a-50deff8538eb/b2c53e19-e42b-4380-a3f5-c04d8b1a12f2"
-					(reference "D38")
+					(reference "D39")
 					(unit 1)
 				)
 				(path "/ce21946f-7655-4864-b48a-50deff8538eb/f5b14127-5321-4517-88f3-03b8eaf90121"
-					(reference "D40")
-					(unit 1)
-				)
+					(reference "D41")
+					(unit 1)
+				)

Commit message: Update SCCS-RPI KiCad design and production files
Split 5V and 3V3 regulation onto dedicated Power sheets with a second
AP64501 buck, extra inductor and passives, update the enclosure
bracket, and regenerate BOM, positions, netlist, gerbers, and
schematics PDF.
Parts:
- renumbered C65 to C53, R91 to R88, R92 to R89, R93 to R90, R94 to R91, U3 to U2
Changed lines of the file:
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@@
 		(dnp no)
 		(fields_autoplaced yes)
-		(property "Reference" "C65"
+		(property "Reference" "C53"
 			(at 102.8763 39.37 90)
 			(show_name no)
@@
 			(project "SCCS-RPI"
 				(path "/ce21946f-7655-4864-b48a-50deff8538eb/67cc456c-a1bb-42f9-9e79-f18883d18275"
-					(reference "C68")
+					(reference "C56")
 					(unit 1)
 				)
 				(path "/ce21946f-7655-4864-b48a-50deff8538eb/6d499a9e-12be-48c7-97b5-aaa8433b7610"
-					(reference "C67")
+					(reference "C55")
 					(unit 1)
 				)
 				(path "/ce21946f-7655-4864-b48a-50deff8538eb/b2c53e19-e42b-4380-a3f5-c04d8b1a12f2"
-					(reference "C65")
+					(reference "C53")
 					(unit 1)
 				)
 				(path "/ce21946f-7655-4864-b48a-50deff8538eb/f5b14127-5321-4517-88f3-03b8eaf90121"
-					(reference "C66")
+					(reference "C54")
 					(unit 1)
 				)
@@
 		(in_pos_files yes)
 		(dnp no)
-		(property "Reference" "R94"
+		(property "Reference" "R91"
 			(at 85.09 63.246 90)
 			(show_name no)
@@
 			(project "SCCS-RPI"
 				(path "/ce21946f-7655-4864-b48a-50deff8538eb/67cc456c-a1bb-42f9-9e79-f18883d18275"
-					(reference "R106")
+					(reference "R103")
 					(unit 1)
 				)
 				(path "/ce21946f-7655-4864-b48a-50deff8538eb/6d499a9e-12be-48c7-97b5-aaa8433b7610"
-					(reference "R102")
+					(reference "R99")
 					(unit 1)
 				)
 				(path "/ce21946f-7655-4864-b48a-50deff8538eb/b2c53e19-e42b-4380-a3f5-c04d8b1a12f2"
-					(reference "R94")
+					(reference "R91")
 					(unit 1)
 				)
 				(path "/ce21946f-7655-4864-b48a-50deff8538eb/f5b14127-5321-4517-88f3-03b8eaf90121"
-					(reference "R98")
+					(reference "R95")
 					(unit 1)
 				)
@@
 		(in_pos_files yes)
 		(dnp no)
-		(property "Reference" "U3"
+		(property "Reference" "U2"
 			(at 70.866 53.34 90)
 			(show_name no)
@@
 			(project "SCCS-RPI"
 				(path "/ce21946f-7655-4864-b48a-50deff8538eb/67cc456c-a1bb-42f9-9e79-f18883d18275"
-					(reference "U6")
+					(reference "U5")
 					(unit 1)
 				)
 				(path "/ce21946f-7655-4864-b48a-50deff8538eb/6d499a9e-12be-48c7-97b5-aaa8433b7610"
-					(reference "U5")
+					(reference "U4")
 					(unit 1)
 				)
 				(path "/ce21946f-7655-4864-b48a-50deff8538eb/b2c53e19-e42b-4380-a3f5-c04d8b1a12f2"
+					(reference "U2")
+					(unit 1)
+				)
+				(path "/ce21946f-7655-4864-b48a-50deff8538eb/f5b14127-5321-4517-88f3-03b8eaf90121"
 					(reference "U3")
-					(unit 1)
-				)
-				(path "/ce21946f-7655-4864-b48a-50deff8538eb/f5b14127-5321-4517-88f3-03b8eaf90121"
-					(reference "U4")
 					(unit 1)
 				)
@@
 		(in_pos_files yes)
 		(dnp no)
-		(property "Reference" "#PWR0112"
+		(property "Reference" "#PWR0111"
 			(at 67.31 64.77 0)
 			(hide yes)
@@
 			(project "SCCS-RPI"
 				(path "/ce21946f-7655-4864-b48a-50deff8538eb/67cc456c-a1bb-42f9-9e79-f18883d18275"
-					(reference "#PWR0121")
+					(reference "#PWR0120")
 					(unit 1)
 				)
 				(path "/ce21946f-7655-4864-b48a-50deff8538eb/6d499a9e-12be-48c7-97b5-aaa8433b7610"
-					(reference "#PWR0118")
+					(reference "#PWR0117")
 					(unit 1)
 				)
 				(path "/ce21946f-7655-4864-b48a-50deff8538eb/b2c53e19-e42b-4380-a3f5-c04d8b1a12f2"
-					(reference "#PWR0112")
+					(reference "#PWR0111")
 					(unit 1)
 				)
 				(path "/ce21946f-7655-4864-b48a-50deff8538eb/f5b14127-5321-4517-88f3-03b8eaf90121"
-					(reference "#PWR0115")
+					(reference "#PWR0114")
 					(unit 1)
 				)
@@
 		(in_pos_files yes)
 		(dnp no)
-		(property "Reference" "R93"
+		(property "Reference" "R90"
 			(at 99.06 56.134 90)
 			(show_name no)
@@
 			(project "SCCS-RPI"
 				(path "/ce21946f-7655-4864-b48a-50deff8538eb/67cc456c-a1bb-42f9-9e79-f18883d18275"
-					(reference "R105")
+					(reference "R102")
 					(unit 1)
 				)
 				(path "/ce21946f-7655-4864-b48a-50deff8538eb/6d499a9e-12be-48c7-97b5-aaa8433b7610"
-					(reference "R101")
+					(reference "R98")
 					(unit 1)
 				)
 				(path "/ce21946f-7655-4864-b48a-50deff8538eb/b2c53e19-e42b-4380-a3f5-c04d8b1a12f2"
-					(reference "R93")
+					(reference "R90")
 					(unit 1)
 				)
 				(path "/ce21946f-7655-4864-b48a-50deff8538eb/f5b14127-5321-4517-88f3-03b8eaf90121"
-					(reference "R97")
+					(reference "R94")
 					(unit 1)
 				)
@@
 		(in_pos_files yes)
 		(dnp no)
-		(property "Reference" "#PWR0111"
+		(property "Reference" "#PWR0110"
 			(at 133.35 46.99 0)
 			(hide yes)
@@
 			(project "SCCS-RPI"
 				(path "/ce21946f-7655-4864-b48a-50deff8538eb/67cc456c-a1bb-42f9-9e79-f18883d18275"
-					(reference "#PWR0120")
+					(reference "#PWR0119")
 					(unit 1)
 				)
 				(path "/ce21946f-7655-4864-b48a-50deff8538eb/6d499a9e-12be-48c7-97b5-aaa8433b7610"
-					(reference "#PWR0117")
+					(reference "#PWR0116")
 					(unit 1)
 				)
 				(path "/ce21946f-7655-4864-b48a-50deff8538eb/b2c53e19-e42b-4380-a3f5-c04d8b1a12f2"
-					(reference "#PWR0111")
+					(reference "#PWR0110")
 					(unit 1)
 				)
 				(path "/ce21946f-7655-4864-b48a-50deff8538eb/f5b14127-5321-4517-88f3-03b8eaf90121"
-					(reference "#PWR0114")
+					(reference "#PWR0113")
 					(unit 1)
 				)
@@
 		(in_pos_files yes)
 		(dnp no)
-		(property "Reference" "R91"
+		(property "Reference" "R88"
 			(at 63.5 48.006 90)
 			(show_name no)
@@
 			(project "SCCS-RPI"
 				(path "/ce21946f-7655-4864-b48a-50deff8538eb/67cc456c-a1bb-42f9-9e79-f18883d18275"
-					(reference "R103")
+					(reference "R100")
 					(unit 1)
 				)
 				(path "/ce21946f-7655-4864-b48a-50deff8538eb/6d499a9e-12be-48c7-97b5-aaa8433b7610"
-					(reference "R99")
+					(reference "R96")
 					(unit 1)
 				)
 				(path "/ce21946f-7655-4864-b48a-50deff8538eb/b2c53e19-e42b-4380-a3f5-c04d8b1a12f2"
-					(reference "R91")
+					(reference "R88")
 					(unit 1)
 				)
 				(path "/ce21946f-7655-4864-b48a-50deff8538eb/f5b14127-5321-4517-88f3-03b8eaf90121"
-					(reference "R95")
+					(reference "R92")
 					(unit 1)
 				)
@@
 		(in_pos_files yes)
 		(dnp no)
-		(property "Reference" "R92"
+		(property "Reference" "R89"
 			(at 121.92 52.578 90)
 			(show_name no)
@@
 			(project "SCCS-RPI"
 				(path "/ce21946f-7655-4864-b48a-50deff8538eb/67cc456c-a1bb-42f9-9e79-f18883d18275"
-					(reference "R104")
+					(reference "R101")
 					(unit 1)
 				)
 				(path "/ce21946f-7655-4864-b48a-50deff8538eb/6d499a9e-12be-48c7-97b5-aaa8433b7610"
-					(reference "R100")
+					(reference "R97")
 					(unit 1)
 				)
 				(path "/ce21946f-7655-4864-b48a-50deff8538eb/b2c53e19-e42b-4380-a3f5-c04d8b1a12f2"
-					(reference "R92")
+					(reference "R89")
 					(unit 1)
 				)
 				(path "/ce21946f-7655-4864-b48a-50deff8538eb/f5b14127-5321-4517-88f3-03b8eaf90121"
-					(reference "R96")
+					(reference "R93")
 					(unit 1)
 				)
@@
 		(in_pos_files yes)
 		(dnp no)
-		(property "Reference" "#PWR0113"
+		(property "Reference" "#PWR0112"
 			(at 91.44 81.28 0)
 			(hide yes)
@@
 			(project "SCCS-RPI"
 				(path "/ce21946f-7655-4864-b48a-50deff8538eb/67cc456c-a1bb-42f9-9e79-f18883d18275"
-					(reference "#PWR0122")
+					(reference "#PWR0121")
 					(unit 1)
 				)
 				(path "/ce21946f-7655-4864-b48a-50deff8538eb/6d499a9e-12be-48c7-97b5-aaa8433b7610"
-					(reference "#PWR0119")
+					(reference "#PWR0118")
 					(unit 1)
 				)
 				(path "/ce21946f-7655-4864-b48a-50deff8538eb/b2c53e19-e42b-4380-a3f5-c04d8b1a12f2"
-					(reference "#PWR0113")
+					(reference "#PWR0112")
 					(unit 1)
 				)
 				(path "/ce21946f-7655-4864-b48a-50deff8538eb/f5b14127-5321-4517-88f3-03b8eaf90121"
-					(reference "#PWR0116")
-					(unit 1)
-				)
+					(reference "#PWR0115")
+					(unit 1)
+				)
